Commit message: Comment SendRosTf and add frame_id input from xacro file

File: urdf/livox_gazebo_sensor.xacro (robot description, xacro)
@@ -9,7 +9,7 @@
     </inertial>
   </xacro:macro>
-  <xacro:macro name="Livox_gazebo_sensor" params="visualize:=True update_rate:=10 resolution:=0.002 noise_mean:=0.0 noise_stddev:=0.01 name:=livox publish_pointcloud_type:=1">
+  <xacro:macro name="Livox_gazebo_sensor" params="visualize:=True update_rate:=10 resolution:=0.002 frame_id:=livox noise_mean:=0.0 noise_stddev:=0.01 name:=livox topic:=pointcloud publish_pointcloud_type:=1">
     <gazebo reference="${name}">
-      <sensor type="ray" name="livox_lidar">
+      <sensor type="ray" name="${name}">
         <pose>0 0 0 0 0 0</pose>
         <visualize>True</visualize>
@@ -43,28 +43,11 @@
           </ray>
           <visualize>${visualize}</visualize>
+          <frame_id>${frame_id}</frame_id>
           <samples>${samples}</samples>
           <downsample>${downsample}</downsample>
           <csv_file_name>${csv_file_name}</csv_file_name>
           <publish_pointcloud_type>${publish_pointcloud_type}</publish_pointcloud_type>
-          <ros_topic>${ros_topic}</ros_topic>
+          <ros_topic>${topic}</ros_topic>
         </plugin>
-      </sensor>
-      <sensor name="livox_imu" type="imu">
-        <always_on>true</always_on>
-        <update_rate>50</update_rate>
-        <visualize>false</visualize>
-        <topic>"/livox/imu"</topic>
-        <plugin filename="libgazebo_ros_imu_sensor.so" name="imu_plugin">
-          <topicName>/livox/imu</topicName>
-          <bodyName>imu_link</bodyName>
-          <updateRateHZ>10.0</updateRateHZ>
-          <xyzOffset>0 0 0</xyzOffset>
-          <!-- <gaussianNoise>0.0026399240948208127</gaussianNoise> -->
-          <gaussianNoise>0.00</gaussianNoise>
-          <rpyOffset>0 0 0</rpyOffset>
-          <frameName>imu_link</frameName>
-          <initialOrientationAsReference>false</initialOrientationAsReference>
-        </plugin>
-        <pose>0 0 0 0 0 0</pose>
       </sensor>
     </gazebo>

File: urdf/livox_mid70.xacro (robot description, xacro)
@@ -11,5 +11,10 @@
   <xacro:property name="csv_file_name" value="package://livox_laser_simulation/scan_mode/mid70.csv"/>
   <xacro:include filename="$(find livox_laser_simulation)/urdf/livox_gazebo_sensor.xacro"/>
-  <xacro:macro name="Livox_Mid70" params="visualize:=True name:=livox publish_pointcloud_type:=0">
+  <xacro:macro name="Livox_Mid70" params="*origin visualize:=True name:=livox topic:=pointcloud parent:=base_link publish_pointcloud_type:=1">
+		<joint name="${name}_base_mount_joint" type="fixed">
+			<xacro:insert_block name="origin" />
+			<parent link="${parent}" />
+			<child link="${name}_base" />
+		</joint>
     <link name="${name}_base">
       <xacro:null_inertial/>
@@ -22,5 +27,5 @@
       </visual>
       <collision>
-          <origin xyz="0 0 0" rpy="0 0 0" />
+          <origin xyz="0.0 0 0.0" rpy="0 0 0" />
           <geometry>
           <mesh filename="package://livox_laser_simulation/meshes/livox_mid40.dae">
@@ -37,5 +42,5 @@
       <origin rpy="0 0 0" xyz="0.0 0.0 0.0"/>
     </joint>
-    <xacro:Livox_gazebo_sensor name="${name}" visualize="${visualize}" publish_pointcloud_type="${publish_pointcloud_type}"/>
+    <xacro:Livox_gazebo_sensor name="${name}" visualize="${visualize}" frame_id="${name}" topic="${topic}" publish_pointcloud_type="${publish_pointcloud_type}"/>
   </xacro:macro>
 </robot>
